File: KiCad/Reloj 3 Placas/Reloj 3 Placas.kicad_pcb (KiCad board)
At the start: 2 copper layers, 233 x 116.8 mm, 81 parts, among them J1 Jack-DC, J2 Conn_2Rows-15Pins, J3 Conn_2Rows-11Pins, J4 Conn_2Rows-15Pins, J5 Conn_2Rows-11Pins, J6 Conn_2Rows-11Pins, J7 Conn_2Rows-11Pins, J8 Conn_2Rows-15Pins, J9 Conn_2Rows-15Pins, Q1 BC548, Q2 BC548, Q3 BC548, Q4 BC548, Q5 BC548, Q6 BC548, Q7 BC548, SW1 SW_SPDT, SW2 SW_Push, SW3 SW_Push, SW4 SW_Push, SW5 SW_Push, U1 74HC14, U2 4050, U3 74HC595

Commit message: Cambio footprint Resistencias y primer ruteo de Displays
Parts:
- R1, R10, R11, R12, R13, R14, R15, R16, R17, R18, R19, R2, R20, R21, R22, R23, R27, R3, R4, R5, R6, R7, R8, R9: footprint Resistor_THT:R_Axial_DIN0204_L3.6mm_D1.6mm_P5.08mm_Horizontal -> Resistor_THT:R_Axial_DIN0204_L3.6mm_D1.6mm_P7.62mm_Horizontal
- moved C4 98.3 mm to (99.8, 135.8), turned to 90 degrees
- moved R8 83.1 mm to (96.6, 138.3), turned to 90 degrees
- moved R7 80.9 mm to (94.2, 138.3), turned to 90 degrees
- moved C3 78.8 mm to (78.0, 146.5)
- moved C2 68.4 mm to (65.9, 146.8)
- moved R5 63.4 mm to (75.4, 141.5)
- moved R6 63.3 mm to (75.4, 143.8)
- moved R3 53.6 mm to (63.2, 141.5)
- moved R4 53.3 mm to (63.2, 143.8)
- moved C1 48.2 mm to (46.8, 135.9), turned to 90 degrees
- moved R2 43.4 mm to (52.0, 138.3), turned to 90 degrees
- moved R1 43.0 mm to (49.8, 138.3), turned to 90 degrees
- moved R15 24.3 mm to (90.7, 112.3), turned to 90 degrees
- moved R16 13.1 mm to (56.9, 112.2), turned to 90 degrees
- moved SW5 3.18 mm to (85.5, 137.8)
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Routing:
- net G: track 0.00 -> 136.1 mm
- net F: track 0.00 -> 122.8 mm, vias 0 -> 10
- net A: track 0.00 -> 119.5 mm, vias 0 -> 10
- net B: track 0.00 -> 102.7 mm, vias 0 -> 10
- net (no net): vias 13 -> 15

Commit message: End design of Display Board.
Parts:
- moved R16 7.19 mm to (59.0, 119.1), turned to -90 degrees
- moved R15 7.14 mm to (92.8, 119.1), turned to -90 degrees
- moved D1 6.58 mm to (89.5, 115.1), turned to 90 degrees
- moved D3 6.54 mm to (55.7, 115.5), turned to 90 degrees
- moved D2 6.41 mm to (89.5, 121.7), turned to 90 degrees
- moved D4 6.32 mm to (55.7, 121.9), turned to 90 degrees
- moved C1 1.06 mm to (47.5, 136.7)
- moved C4 1.06 mm to (100.5, 136.5)
- moved R1 1.06 mm to (50.5, 139.1)
- moved R2 1.06 mm to (52.8, 139.1)
- moved R7 1.06 mm to (95.0, 139.1)
- moved R8 1.06 mm to (97.3, 139.1)
- moved SW2 1.06 mm to (56.8, 138.5)
- moved SW3 1.06 mm to (66.5, 138.5)
- moved SW4 1.06 mm to (76.5, 138.5)
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Routing:
- net D: track 0.00 -> 151.1 mm, vias 0 -> 12
- net SEL 1: track 0.00 -> 146.0 mm, vias 0 -> 1
- net E: track 0.00 -> 144.9 mm, vias 0 -> 4
- net C: track 0.00 -> 131.9 mm, vias 0 -> 8
- net 3,3V: track 0.00 -> 111.6 mm
- net SEL 2: track 0.00 -> 86.5 mm, vias 0 -> 3
- net GND: track 0.00 -> 78.2 mm
- net A: track 119.5 -> 193.9 mm
- net MODE: track 0.00 -> 61.4 mm
- net SEL 3: track 0.00 -> 57.3 mm
- net B: track 102.7 -> 158.7 mm
- net G: track 136.1 -> 187.6 mm, vias 0 -> 2
- net F: track 122.8 -> 168.6 mm, vias 10 -> 11
- net INC: track 0.00 -> 44.0 mm
- net SEL 4: track 0.00 -> 40.6 mm
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